Commit message: Se agregaron otros 2 brazos, funcionando

File: install/modelrobot_pkg_g07/share/modelrobot_pkg_g07/model/MS3R.urdf.xacro (robot description, xacro)
@@ -74,5 +74,5 @@
         <parent link="soporte_link"/>
         <child link="brazo1_link"/>
-        <origin xyz="0 0 ${blz}" rpy="0 0 0"/>
+        <origin xyz="${-plx/2} 0 ${blz}" rpy="0 0 0"/>
     </joint>
     <xacro:brazo_macro p_name ="brazo1_link"
@@ -80,3 +80,29 @@
                        p_ly="${ply}"
                        p_lz="${plz}"/>
+    <joint name="brazo1_brazo2_joint" type="continuous">
+    <!-- ... -->
+        <parent link="brazo1_link"/>
+        <child link="brazo2_link"/>
+        <origin xyz="${-plx} 0 ${plz - 2*blz}" rpy="0 0 0"/>
+        <axis xyz="1 0 0"/>
+        <limit effort="1" lower="0" upper="${2*pi}" velocity="1"/>
+        <dynamics damping="1" friction="1"/>
+    </joint>
+    <xacro:brazo_macro p_name ="brazo2_link"
+                       p_lx="${plx}"
+                       p_ly="${ply}"
+                       p_lz="${plz}"/>
+    <joint name="brazo2_brazo3_joint" type="continuous">
+    <!-- ... -->
+        <parent link="brazo2_link"/>
+        <child link="brazo3_link"/>
+        <origin xyz="${plx} 0 ${plz - 2*blz}" rpy="0 0 0"/>
+        <axis xyz="1 0 0"/>
+        <limit effort="1" lower="0" upper="${2*pi}" velocity="1"/>
+        <dynamics damping="1" friction="1"/>
+    </joint>
+    <xacro:brazo_macro p_name ="brazo3_link"
+                       p_lx="${plx}"
+                       p_ly="${ply}"
+                       p_lz="${plz}"/>
 </robot>

Commit message: Version con los archivos stl, no funcionando

File: install/modelrobot_pkg_g07/share/modelrobot_pkg_g07/model/MS3R.urdf.xacro (robot description, xacro)
@@ -106,3 +106,34 @@
                        p_ly="${ply}"
                        p_lz="${plz}"/>
+    <joint name="brazo3_brazo4_joint" type="continuous">
+    <!-- ... -->
+        <parent link="brazo3_link"/>
+        <child link="brazo4_link"/>
+        <origin xyz="${plx} 0 ${plz - 2*blz}" rpy="0 0 0"/>
+        <axis xyz="1 0 0"/>
+        <limit effort="1" lower="0" upper="${2*pi}" velocity="1"/>
+        <dynamics damping="1" friction="1"/>
+    </joint>
+    <link name="brazo4">
+        <!-- ... -->
+        <visual>
+        <!-- ... -->
+            <geometry>
+                <mesh filename="package://model/Cuerpo1.stl" scale="0.1 0.1 0.1"/>
+            </geometry>
+            <origin xyz="${plx/2} 0 ${plz/2-blz}" rpy="0 0 0"/>
+            <inertial>
+            <!-- ... -->
+                <mass value="1"/>
+                <origin xyz="0 0 0" rpy="0 0 0"/>
+                <inertia ixx="1.69" ixy="0" ixz="0" iyy="3.125" iyz="0" izz="1.69"/>
+            </inertial>
+            <collision>
+            <!-- ... -->
+                <geometry>
+                    <mesh filename="package://model/Cuerpo1.stl" scale="0.1 0.1 0.1"/>
+                </geometry>
+                <origin xyz="${plx/2} 0 ${plz/2-blz}" rpy="0 0 0"/>
+            </collision>
+    </link>
 </robot>
